Commit message: Missile reward redesign, drop flashnet PPO, env and tooling fixes

File: environments/common/original_pyflyt/models/vehicles/quadplane/quadplane.urdf (robot description, URDF)
Before this commit: robot quadplane, 12 links, 11 joints
Links:
- link base_link: geometry collision box size=0.1 0.2 0.2
Joints:
- joint ail_left_joint: origin xyz=-0.95 -0.5 0 rpy=0 0 0 -> xyz=-0.5 0.95 0 rpy=0 0 -1.5707963267948966
- joint ail_right_joint: origin xyz=0.95 -0.5  0 rpy=0 0 0 -> xyz=-0.5 -0.95 0 rpy=0 0 -1.5707963267948966
- joint fuselage_joint: origin xyz=0 -0.45 0 rpy=0 0 0 -> xyz=-0.45 0 0 rpy=0 0 -1.5707963267948966
- joint horizontal_tail_joint: origin xyz=0 -1.1 0 rpy=0 0 0 -> xyz=-1.1 0 0 rpy=0 0 -1.5707963267948966
- joint main_wing_joint: origin xyz=0 -0.5 0 rpy=0 0 0 -> xyz=-0.5 0 0 rpy=0 0 -1.5707963267948966
- joint motor_joint: origin xyz=0 0 0 rpy=0 0 0 -> xyz=0 0 0 rpy=0 0 -1.5707963267948966
- joint prop1_joint: origin xyz=0.5 0.05 0 rpy=0 0 0 -> xyz=0.05 -0.5 0 rpy=0 0 -1.5707963267948966
- joint prop2_joint: origin xyz=-0.5 -0.95 0 rpy=0 0 0 -> xyz=-0.95 0.5 0 rpy=0 0 -1.5707963267948966
- joint prop3_joint: origin xyz=-0.5 0.05 0 rpy=0 0 0 -> xyz=0.05 0.5 0 rpy=0 0 -1.5707963267948966
- joint prop4_joint: origin xyz=0.5 -0.95 0 rpy=0 0 0 -> xyz=-0.95 -0.5 0 rpy=0 0 -1.5707963267948966
- joint vertical_tail_joint: origin xyz=0 -1.1 0.15 rpy=0 0 0 -> xyz=-1.1 0 0.15 rpy=0 0 -1.5707963267948966
